File: TS100C.sch (KiCad schematic (older format))
At the start: 51 parts, among them J1 USB-C_Power, J2 OLED_64x32, J3 A, J4 B, P1 TC2030-CTX, Q1 SS8050, Q2 DMP3017SFG, SW1 Setup, U1 USBLC6-2SC6, U2 AP2204R-3.3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

Commit message: added most parts
Parts:
- added C18: 0.1μF, Capacitor_SMD:C_0402_1005Metric, symbol Device:C
- added R18: 1k, Resistor_SMD:R_0402_1005Metric, symbol Device:R
- added R19: 20, Resistor_SMD:R_0402_1005Metric, symbol Device:R
- added SW2: key2, Button_Switch_SMD:SW_SPST_TL3305B, symbol Switch:SW_Push
- added U6: MCP9700AT-ETT, Package_TO_SOT_SMD:SOT-23, symbol Sensor_Temperature:MCP9700AT-ETT
- C16: value 10n -> 0.1uF
- C17: value 100n -> 0.1μF
- Q2: footprint Package_SON:Diodes_PowerDI3333-8 -> otter:Diodes_PowerDI3333-8
- SW1: value Setup -> key1; footprint Button_Switch_SMD:SW_SPST_EVQP7C -> Button_Switch_SMD:SW_SPST_TL3305B
Connections:
- wire segments 181 -> 190
Other:
- note added: "Buttons\nTagConnect\nDisplay\nOtter <3"
- note added: "todo"
- moved on the sheet: C16, C17, D1, D3, J3, J4, Q1, R12, R14, R15, R16, R17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

Commit message: update PCB
Parts:
- J1: symbol otter:USB-C_Power -> TS100C-rescue:USB-C_Power-otter
- J2: footprint Connector_Harwin:Harwin_M20-89014xx_1x14_P2.54mm_Horizontal -> otter:0.69OLED
- P1: symbol usb-c-otter-rescue:TC2030-CTX-Tag-Connect-pd-buddy-sink-rescue-usb-c-otter-rescue -> TS100C-rescue:TC2030-CTX-Tag-Connect-pd-buddy-sink-rescue-usb-c-otter-rescue-usb-c-otter-rescue
- Q2: symbol usb-c-otter-rescue:DMP3017SFG-pd-buddy-pd-buddy-sink-rescue-pd-buddy-sink-rescue-usb-c-otter-rescue -> TS100C-rescue:DMP3017SFG-pd-buddy-pd-buddy-sink-rescue-pd-buddy-sink-rescue-usb-c-otter-rescue-usb-c-otter-rescue
Changed lines of the file:
@@
 EESchema Schematic File Version 4
-LIBS:usb-c-otter-cache
+LIBS:TS100C-cache
 EELAYER 26 0
 EELAYER END
@@
 OUT
 $Comp
-L usb-c-otter-rescue:DMP3017SFG-pd-buddy-pd-buddy-sink-rescue-pd-buddy-sink-rescue-usb-c-otter-rescue Q?
+L TS100C-rescue:DMP3017SFG-pd-buddy-pd-buddy-sink-rescue-pd-buddy-sink-rescue-usb-c-otter-rescue-usb-c-otter-rescue Q?
 U 1 1 5BD78C00
 P 14700 2200
@@
 	9200 3800 9200 4000
 $Comp
-L usb-c-otter-rescue:TC2030-CTX-Tag-Connect-pd-buddy-sink-rescue-usb-c-otter-rescue P1
+L TS100C-rescue:TC2030-CTX-Tag-Connect-pd-buddy-sink-rescue-usb-c-otter-rescue-usb-c-otter-rescue P1
 U 1 1 5BE3611C
 P 1900 3850
@@
 F 0 "J2" H 14230 7092 50  0000 L CNN
 F 1 "OLED_64x32" H 14230 7001 50  0000 L CNN
-F 2 "Connector_Harwin:Harwin_M20-89014xx_1x14_P2.54mm_Horizontal" H 14150 7100 50  0001 C CNN
+F 2 "otter:0.69OLED" H 14150 7100 50  0001 C CNN
 F 3 "~" H 14150 7100 50  0001 C CNN
 	1    14150 7100
@@
 CC2_P
 $Comp
-L otter:USB-C_Power J1
+L TS100C-rescue:USB-C_Power-otter J1
 U 1 1 5BF68277
 P 1000 2550

Commit message: update PCB
Parts:
- removed C6: 0.1μF, Capacitor_SMD:C_0402_1005Metric, symbol Device:C
- removed D1: Status, LED_SMD:LED_0603_1608Metric, symbol Device:LED
- removed D2: Power, LED_SMD:LED_0603_1608Metric, symbol Device:LED
- removed J1: USB-C_Power, otter:USB-C_Power, symbol TS100C-rescue:USB-C_Power-otter
- removed JP1: Boot, Jumper:SolderJumper-2_P1.3mm_Open_RoundedPad1.0x1.5mm, symbol Jumper:SolderJumper_2_Open
- removed R7, R8: 2k, Resistor_SMD:R_0402_1005Metric, symbol Device:R
- added J1: USB_C, Connector_USB:USB_C_Receptacle_Amphenol_12401548E4-2A, symbol usb-c-otter-rescue:USB_C_Receptacle-Connector-pd-buddy-sink-rescue-pd-buddy-sin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
- added J5: DNP, Resistor_SMD:R_0402_1005Metric, symbol Device:R
- SW1, SW2: footprint Button_Switch_SMD:SW_SPST_TL3305B -> Button_Switch_SMD:SW_SPST_PTS810
- U1: value USBLC6-2SC6 -> USBLC6-4SC6
Connections:
- net labels added: USB_N, USB_P
- net labels removed: CC1_P, CC2_P
- wire segments 190 -> 200
Other:
- note removed: "Buttons\nTagConnect\nDisplay\nOtter <3"
- note removed: "todo"
- moved on the sheet: C18, P1, U1, U3

Commit message: update PCB
Parts:
- added C6: 0.1μF, Capacitor_SMD:C_0402_1005Metric, symbol Device:C
Changed lines of the file:
@@
 	-1   0    0    1
 $EndComp
+$Comp
+L Device:C C6
+U 1 1 5A9C1A0C
+P 4650 5150
+F 0 "C6" H 4765 5196 50  0000 L CNN
+F 1 "0.1μF" H 4765 5105 50  0000 L CNN
+F 2 "Capacitor_SMD:C_0402_1005Metric" H 4688 5000 50  0001 C CNN
+F 3 "~" H 4650 5150 50  0001 C CNN
+	1    4650 5150
+	1    0    0    -1
+$EndComp
 $EndSCHEMATC

Commit message: fixed connector error
Changed lines of the file:
@@
 L power:GND #PWR0136
 U 1 1 5C00E02C
-P 11950 3450
-F 0 "#PWR0136" H 11950 3200 50  0001 C CNN
-F 1 "GND" H 11955 3277 50  0000 C CNN
-F 2 "" H 11950 3450 50  0001 C CNN
-F 3 "" H 11950 3450 50  0001 C CNN
-	1    11950 3450
-	1    0    0    -1
+P 11950 2850
+F 0 "#PWR0136" H 11950 2600 50  0001 C CNN
+F 1 "GND" H 11955 2677 50  0000 C CNN
+F 2 "" H 11950 2850 50  0001 C CNN
+F 3 "" H 11950 2850 50  0001 C CNN
+	1    11950 2850
+	-1   0    0    1
 $EndComp
 $Comp
@@
 L power:+3V3 #PWR0137
 U 1 1 5C03FC4A
-P 11950 2850
-F 0 "#PWR0137" H 11950 2700 50  0001 C CNN
-F 1 "+3V3" H 11965 3023 50  0000 C CNN
-F 2 "" H 11950 2850 50  0001 C CNN
-F 3 "" H 11950 2850 50  0001 C CNN
-	1    11950 2850
-	1    0    0    -1
+P 11950 3450
+F 0 "#PWR0137" H 11950 3300 50  0001 C CNN
+F 1 "+3V3" H 11965 3623 50  0000 C CNN
+F 2 "" H 11950 3450 50  0001 C CNN
+F 3 "" H 11950 3450 50  0001 C CNN
+	1    11950 3450
+	-1   0    0    1
 $EndComp
 Text GLabel 10850 2400 0    60   Input ~ 0

Commit message: update PCB
Parts:
- J4: footprint otter:Keystone_3621 -> otter:3622TR
Changed lines of the file:
@@
 F 0 "J4" H 15528 3026 50  0000 L CNN
 F 1 "B" H 15528 2935 50  0000 L CNN
-F 2 "otter:Keystone_3621" H 15500 3000 50  0001 C CNN
+F 2 "otter:3622TR" H 15500 3000 50  0001 C CNN
 F 3 "~" H 15500 3000 50  0001 C CNN
 	1    15500 3000

Commit message: update pcb
Parts:
- J5: footprint Resistor_SMD:R_0402_1005Metric -> Jumper:SolderJumper-2_P1.3mm_Open_RoundedPad1.0x1.5mm
Changed lines of the file:
@@
 F 0 "J5" H 5680 1304 50  0000 R CNN
 F 1 "DNP" H 5680 1395 50  0000 R CNN
-F 2 "Resistor_SMD:R_0402_1005Metric" V 5680 1350 50  0001 C CNN
+F 2 "Jumper:SolderJumper-2_P1.3mm_Open_RoundedPad1.0x1.5mm" V 5680 1350 50  0001 C CNN
 F 3 "~" H 5750 1350 50  0001 C CNN
 	1    5750 1350
