File: KiCAD/TS100C.sch (KiCad schematic (older format))
At the start: 52 parts, among them J1 USB_C, J2 OLED_64x32, J3 A, J4 B, J5 DNP, P1 TC2030-CTX, Q1 SS8050, Q2 DMP3017SFG, SW1 key1, SW2 key2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

Commit message: updated PCB+schematic to STUSB4500
Parts:
- removed J1: USB_C, Connector_USB:USB_C_Receptacle_Amphenol_12401548E4-2A, symbol usb-c-otter-rescue:USB_C_Receptacle-Connector-pd-buddy-sink-rescue-pd-buddy-sin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
- removed U3: FUSB302BMPX, Package_DFN_QFN:WQFN-14-1EP_2.5x2.5mm_P0.5mm_EP1.45x1.45mm, symbol Interface_USB:FUSB302BMPX
- added C19, C20, C21: 0.1μF, Capacitor_SMD:C_0402_1005Metric, symbol Device:C
- added C22: 0.1μF, Capacitor_SMD:C_0402_1005Metric, symbol Device:C_Small
- added J1: USB_C_Receptacle_USB2.0, otter:USB-C 16Pin, symbol Connector:USB_C_Receptacle_USB2.0
- added R20, R21: 33, Resistor_SMD:R_0402_1005Metric, symbol Device:R
- added R22: 10m, Resistor_SMD:R_0805_2012Metric, symbol Device:R_Small
- added R7: 2kΩ, Resistor_SMD:R_0402_1005Metric, symbol Device:R
- added R8: 2k, Resistor_SMD:R_0402_1005Metric, symbol Device:R_Small
- added U3: STUSB4500, Package_DFN_QFN:QFN-24-1EP_4x4mm_P0.5mm_EP2.7x2.7mm, symbol otter:STUSB4500
- added U7: SI8540, Package_TO_SOT_SMD:SOT-23-5, symbol otter:SI8540
- D3: footprint Diode_SMD:D_SMA -> Diode_SMD:D_SOD-123F
- J5: footprint Jumper:SolderJumper-2_P1.3mm_Open_RoundedPad1.0x1.5mm -> Resistor_SMD:R_0402_1005Metric
Connections:
- net labels added: IIN, SW1
- wire segments 200 -> 198
- no-connect marks 0 -> 10
Other:
- moved on the sheet: C16, C17, C18, D3, J3, J4, Q1, Q2, R12, R14, R15, R16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

Commit message: updated pcb
Parts:
- added R?: 2kΩ, Resistor_SMD:R_0402_1005Metric, symbol Device:R
Connections:
- net VBUS: now also R?.2
- net at U3.18 (VBUS_VS_DISCH): now also R?.1
- no-connect marks 10 -> 9
Changed lines of the file:
@@
 NoConn ~ 5100 7900
 NoConn ~ 5100 8000
-NoConn ~ 3500 7550
 NoConn ~ 3500 8250
 NoConn ~ 3500 8350
@@
 Text GLabel 12550 2100 0    50   Input ~ 0
 IIN
+$Comp
+L Device:R R?
+U 1 1 5D2E68C3
+P 3350 7400
+F 0 "R?" H 3419 7446 50  0000 L CNN
+F 1 "2kΩ" H 3419 7355 50  0000 L CNN
+F 2 "Resistor_SMD:R_0402_1005Metric" V 3280 7400 50  0001 C CNN
+F 3 "~" H 3350 7400 50  0001 C CNN
+	1    3350 7400
+	-1   0    0    1
+$EndComp
+$Comp
+L power:VBUS #PWR?
+U 1 1 5D2F1212
+P 3350 7200
+AR Path="/588FB1D7/5D2F1212" Ref="#PWR?"  Part="1"
+AR Path="/588FD270/5D2F1212" Ref="#PWR?"  Part="1"
+AR Path="/5D2F1212" Ref="#PWR?"  Part="1"
+F 0 "#PWR?" H 3350 7050 50  0001 C CNN
+F 1 "VBUS" H 3365 7373 50  0000 C CNN
+F 2 "" H 3350 7200 50  0001 C CNN
+F 3 "" H 3350 7200 50  0001 C CNN
+	1    3350 7200
+	1    0    0    -1
+$EndComp
+Wire Wire Line
+	3350 7250 3350 7200
+Wire Wire Line
+	3350 7550 3500 7550
 $EndSCHEMATC

Commit message: updated hardware
Parts:
- gave numbers to parts that had none: 1
Connections:
- net GND: now also U3.12 (ADDR0), U3.13 (ADDR1)
- no-connect marks 9 -> 7
Changed lines of the file:
@@
 NoConn ~ 5100 7900
 NoConn ~ 5100 8000
-NoConn ~ 3500 8250
-NoConn ~ 3500 8350
 $Comp
 L power:GND #PWR0116
@@
 IIN
 $Comp
-L Device:R R?
+L Device:R R23
 U 1 1 5D2E68C3
 P 3350 7400
-F 0 "R?" H 3419 7446 50  0000 L CNN
+F 0 "R23" H 3419 7446 50  0000 L CNN
 F 1 "2kΩ" H 3419 7355 50  0000 L CNN
 F 2 "Resistor_SMD:R_0402_1005Metric" V 3280 7400 50  0001 C CNN
@@
 AR Path="/588FB1D7/5D2F1212" Ref="#PWR?"  Part="1"
 AR Path="/588FD270/5D2F1212" Ref="#PWR?"  Part="1"
-AR Path="/5D2F1212" Ref="#PWR?"  Part="1"
-F 0 "#PWR?" H 3350 7050 50  0001 C CNN
+AR Path="/5D2F1212" Ref="#PWR0146"  Part="1"
+F 0 "#PWR0146" H 3350 7050 50  0001 C CNN
 F 1 "VBUS" H 3365 7373 50  0000 C CNN
 F 2 "" H 3350 7200 50  0001 C CNN
@@
 Wire Wire Line
 	3350 7550 3500 7550
+Wire Wire Line
+	3450 8250 3500 8250
+Wire Wire Line
+	3500 8250 3500 8350
+$Comp
+L power:GND #PWR?
+U 1 1 5D391174
+P 3450 8250
+F 0 "#PWR?" H 3450 8000 50  0001 C CNN
+F 1 "GND" H 3455 8077 50  0000 C CNN
+F 2 "" H 3450 8250 50  0001 C CNN
+F 3 "" H 3450 8250 50  0001 C CNN
+	1    3450 8250
+	0    1    1    0
+$EndComp
+Connection ~ 3500 8250
 $EndSCHEMATC

Commit message: added todos
Parts:
- C16: value 0.1uF -> 100p
Connections:
- net PWM: now also U4.29 (PA8); no longer U4.39 (PB3)
Other:
- note added: "Todo:\nDesign auf 4/4 mil\nvias kleiner\nTimer umpfoten"
Changed lines of the file:
@@
 Text GLabel 13000 4050 0    60   Input ~ 0
-PWM
-Text GLabel 6700 2800 0    60   Input ~ 0
 PWM
 Text GLabel 5100 3500 0    60   Input ~ 0
@@
 OLED_PULLUP
 Wire Wire Line
-	6700 2800 6750 2800
-Wire Wire Line
 	6750 3100 6700 3100
 Wire Wire Line
@@
 P 11500 3950
 F 0 "C16" V 11450 3850 50  0000 C CNN
-F 1 "0.1uF" V 11600 3950 50  0000 C CNN
+F 1 "100p" V 11600 3950 50  0000 C CNN
 F 2 "Capacitor_SMD:C_0402_1005Metric" H 11500 3950 50  0001 C CNN
 F 3 "~" H 11500 3950 50  0001 C CNN
@@
 	3500 8250 3500 8350
 $Comp
-L power:GND #PWR?
+L power:GND #PWR0147
 U 1 1 5D391174
 P 3450 8250
-F 0 "#PWR?" H 3450 8000 50  0001 C CNN
+F 0 "#PWR0147" H 3450 8000 50  0001 C CNN
 F 1 "GND" H 3455 8077 50  0000 C CNN
 F 2 "" H 3450 8250 50  0001 C CNN
@@
 $EndComp
 Connection ~ 3500 8250
+Text GLabel 8050 3300 2    60   Input ~ 0
+PWM
+Text Notes 9450 3600 0    50   ~ 0
+Todo:\nDesign auf 4/4 mil\nvias kleiner\nTimer umpfoten
 $EndSCHEMATC

Commit message: fixed bom
Parts:
- C1: value 1.0μF 25V -> 1μF 25V
- C11, C9: value 1μF -> 1μF 25V
- C16: value 100p -> TBD (18p)
- C17: value 0.1μF -> TBD (100n)
- C4: value 2.2μF -> 1μF 25V
- R10, R13, R5, R8, R9: value 2k -> 2k37
- R12: value 10k -> 2k37
- R14, R18: value 1k -> 2k37
- R23, R3, R4, R6, R7: value 2kΩ -> 2k37
Connections:
- net +3V3: now also R10.2, R13.2
- removed net OLED_PULLUP: R10.2, R13.2, U4.45 (PB8)
- net SW1: no longer names the net of J5.1, R5.2, U4.44 (BOOT0)
- net SW1: no longer SW1.2, U4.13 (PA3)
- new net: SW1.2, U4.13 (PA3)
Changed lines of the file:
@@
 EESchema Schematic File Version 4
 LIBS:TS100C-cache
-EELAYER 29 0
+EELAYER 26 0
 EELAYER END
 $Descr A3 16535 11693
@@
 Connection ~ 5200 3000
 Wire Wire Line
-	6700 3300 6750 3300
-Wire Wire Line
 	8050 3800 8350 3800
 Wire Wire Line
@@
 P 5750 1850
 F 0 "R5" H 5680 1804 50  0000 R CNN
-F 1 "2k" H 5680 1895 50  0000 R CNN
+F 1 "2k37" H 5680 1895 50  0000 R CNN
 F 2 "Resistor_SMD:R_0402_1005Metric" V 5680 1850 50  0001 C CNN
 F 3 "~" H 5750 1850 50  0001 C CNN
@@
 P 5200 3250
 F 0 "R3" H 5269 3296 50  0000 L CNN
-F 1 "2kΩ" H 5269 3205 50  0000 L CNN
+F 1 "2k37" H 5269 3205 50  0000 L CNN
 F 2 "Resistor_SMD:R_0402_1005Metric" V 5130 3250 50  0001 C CNN
 F 3 "~" H 5200 3250 50  0001 C CNN
@@
 P 5500 3250
 F 0 "R4" H 5569 3296 50  0000 L CNN
-F 1 "2kΩ" H 5569 3205 50  0000 L CNN
+F 1 "2k37" H 5569 3205 50  0000 L CNN
 F 2 "Resistor_SMD:R_0402_1005Metric" V 5430 3250 50  0001 C CNN
 F 3 "~" H 5500 3250 50  0001 C CNN
@@
 P 5800 3250
 F 0 "R6" H 5869 3296 50  0000 L CNN
-F 1 "2kΩ" H 5869 3205 50  0000 L CNN
+F 1 "2k37" H 5869 3205 50  0000 L CNN
 F 2 "Resistor_SMD:R_0402_1005Metric" V 5730 3250 50  0001 C CNN
 F 3 "~" H 5800 3250 50  0001 C CNN
@@
 U 1 1 5A9C1ACC
 P 5150 5150
-F 0 "C7" H 5035 5104 50  0000 R CNN
-F 1 "0.1μF" H 5035 5195 50  0000 R CNN
+F 0 "C7" H 5035 5196 50  0000 R CNN
+F 1 "0.1μF" H 5035 5105 50  0000 R CNN
 F 2 "Capacitor_SMD:C_0402_1005Metric" H 5188 5000 50  0001 C CNN
 F 3 "~" H 5150 5150 50  0001 C CNN
@@
 P 6150 5150
 F 0 "C9" H 6265 5196 50  0000 L CNN
-F 1 "1μF" H 6265 5105 50  0000 L CNN
+F 1 "1μF 25V" H 6265 5105 50  0000 L CNN
 F 2 "Capacitor_SMD:C_0603_1608Metric" H 6188 5000 50  0001 C CNN
 F 3 "~" H 6150 5150 50  0001 C CNN
@@
 AR Path="/5BD75E6E" Ref="C1"  Part="1"
 F 0 "C1" H 3515 1496 50  0000 L CNN
-F 1 "1.0μF 25V" H 3515 1405 50  0000 L CNN
+F 1 "1μF 25V" H 3515 1405 50  0000 L CNN
 F 2 "Capacitor_SMD:C_0603_1608Metric" H 3438 1300 50  0001 C CNN
 F 3 "~" H 3400 1450 50  0001 C CNN
@@
 AR Path="/5BD75E75" Ref="C4"  Part="1"
 F 0 "C4" H 4715 1496 50  0000 L CNN
-F 1 "2.2μF" H 4715 1405 50  0000 L CNN
+F 1 "1μF 25V" H 4715 1405 50  0000 L CNN
 F 2 "Capacitor_SMD:C_0603_1608Metric" H 4638 1300 50  0001 C CNN
 F 3 "~" H 4600 1450 50  0001 C CNN
@@
 AR Path="/5BD78C38" Ref="R12"  Part="1"
 F 0 "R12" H 13670 3346 50  0000 L CNN
-F 1 "10k" H 13670 3255 50  0000 L CNN
+F 1 "2k37" H 13670 3255 50  0000 L CNN
 F 2 "Resistor_SMD:R_0402_1005Metric" V 13530 3300 50  0001 C CNN
 F 3 "~" H 13600 3300 50  0001 C CNN
@@
 AR Path="/5BD78C3F" Ref="R9"  Part="1"
 F 0 "R9" V 12943 4050 50  0000 C CNN
-F 1 "2k" V 13034 4050 50  0000 C CNN
+F 1 "2k37" V 13034 4050 50  0000 C CNN
 F 2 "Resistor_SMD:R_0402_1005Metric" V 13080 4050 50  0001 C CNN
 F 3 "~" H 13150 4050 50  0001 C CNN
@@
 AR Path="/5BD7CA3C" Ref="C11"  Part="1"
 F 0 "C11" H 7215 5196 50  0000 L CNN
-F 1 "1μF" H 7215 5105 50  0000 L CNN
+F 1 "1μF 25V" H 7215 5105 50  0000 L CNN
 F 2 "Capacitor_SMD:C_0603_1608Metric" H 7138 5000 50  0001 C CNN
 F 3 "~" H 7100 5150 50  0001 C CNN
@@
 Text GLabel 3400 7950 0    60   Input ~ 0
 CC2
-Text GLabel 2150 2450 2    60   Input ~ 0
-CC1
-Text GLabel 2150 2550 2    60   Input ~ 0
-CC2
 Text GLabel 2950 3450 0    46   Input ~ 0
 USB_N
@@
 Wire Wire Line
 	13300 6900 13300 7000
-Wire Wire Line
-	13000 6800 13000 6900
 Connection ~ 13000 6900
 Wire Wire Line
@@
 P 13000 7150
 F 0 "R10" H 13069 7196 50  0000 L CNN
-F 1 "2k" H 13069 7105 50  0000 L CNN
+F 1 "2k37" H 13069 7105 50  0000 L CNN
 F 2 "Resistor_SMD:R_0402_1005Metric" V 12930 7150 50  0001 C CNN
 F 3 "~" H 13000 7150 50  0001 C CNN
@@
 P 13300 7150
 F 0 "R13" H 13369 7196 50  0000 L CNN
-F 1 "2k" H 13369 7105 50  0000 L CNN
+F 1 "2k37" H 13369 7105 50  0000 L CNN
 F 2 "Resistor_SMD:R_0402_1005Metric" V 13230 7150 50  0001 C CNN
 F 3 "~" H 13300 7150 50  0001 C CNN
@@
 Text GLabel 6700 3200 0    60   Input ~ 0
 OLED_SDA
-Text GLabel 13000 6800 0    60   Input ~ 0
-OLED_PULLUP
-Text GLabel 6700 3300 0    60   Input ~ 0
-OLED_PULLUP
 Wire Wire Line
 	6750 3100 6700 3100
@@
 P 12550 4500
 F 0 "C17" H 12642 4546 50  0000 L CNN
-F 1 "0.1μF" H 12642 4455 50  0000 L CNN
+F 1 "TBD (100n)" H 12642 4455 50  0000 L CNN
 F 2 "Capacitor_SMD:C_0402_1005Metric" H 12550 4500 50  0001 C CNN
 F 3 "~" H 12550 4500 50  0001 C CNN
@@
 P 11500 3950
 F 0 "C16" V 11450 3850 50  0000 C CNN
-F 1 "100p" V 11600 3950 50  0000 C CNN
+F 1 "TBD (18p)" V 11600 3950 50  0000 C CNN
 F 2 "Capacitor_SMD:C_0402_1005Metric" H 11500 3950 50  0001 C CNN
 F 3 "~" H 11500 3950 50  0001 C CNN
@@
 P 10850 3750
 F 0 "R14" V 10643 3750 50  0000 C CNN
-F 1 "1k" V 10850 3750 50  0000 C CNN
+F 1 "2k37" V 10734 3750 50  0000 C CNN
 F 2 "Resistor_SMD:R_0402_1005Metric" V 10780 3750 50  0001 C CNN
 F 3 "~" H 10850 3750 50  0001 C CNN
@@
 P 11150 7450
 F 0 "R18" V 10943 7450 50  0000 C CNN
-F 1 "1k" V 11150 7450 50  0000 C CNN
+F 1 "2k37" V 11034 7450 50  0000 C CNN
 F 2 "Resistor_SMD:R_0402_1005Metric" V 11080 7450 50  0001 C CNN
 F 3 "~" H 11150 7450 50  0001 C CNN
@@
 P 5250 8550
 F 0 "R7" H 5319 8596 50  0000 L CNN
-F 1 "2kΩ" H 5319 8505 50  0000 L CNN
+F 1 "2k37" H 5319 8505 50  0000 L CNN
 F 2 "Resistor_SMD:R_0402_1005Metric" V 5180 8550 50  0001 C CNN
 F 3 "~" H 5250 8550 50  0001 C CNN
@@
 P 13050 2200
 F 0 "R8" H 13109 2246 50  0000 L CNN
-F 1 "2k" H 13109 2155 50  0000 L CNN
+F 1 "2k37" H 13109 2155 50  0000 L CNN
 F 2 "Resistor_SMD:R_0402_1005Metric" H 13050 2200 50  0001 C CNN
 F 3 "~" H 13050 2200 50  0001 C CNN
@@
 	1    0    0    -1
 $EndComp
-Text GLabel 9000 2800 1    50   Input ~ 0
-SW1
-Text GLabel 5750 1600 0    50   Input ~ 0
-SW1
 Text GLabel 8350 2500 2    50   Input ~ 0
 IIN
@@
 P 3350 7400
 F 0 "R23" H 3419 7446 50  0000 L CNN
-F 1 "2kΩ" H 3419 7355 50  0000 L CNN
+F 1 "2k37" H 3419 7355 50  0000 L CNN
 F 2 "Resistor_SMD:R_0402_1005Metric" V 3280 7400 50  0001 C CNN
 F 3 "~" H 3350 7400 50  0001 C CNN
@@
 Text Notes 9450 3600 0    50   ~ 0
 Todo:\nDesign auf 4/4 mil\nvias kleiner\nTimer umpfoten
+$Comp
+L power:+3V3 #PWR0148
+U 1 1 5D3A56D4
+P 13000 6700
+F 0 "#PWR0148" H 13000 6550 50  0001 C CNN
+F 1 "+3V3" H 13015 6873 50  0000 C CNN
+F 2 "" H 13000 6700 50  0001 C CNN
+F 3 "" H 13000 6700 50  0001 C CNN
+	1    13000 6700
+	1    0    0    -1
+$EndComp
+Wire Wire Line
+	13000 6700 13000 6900
+Text GLabel 2150 2450 2    60   Input ~ 0
+CC1
+Text GLabel 2150 2550 2    60   Input ~ 0
+CC2
 $EndSCHEMATC

Commit message: optimized bom
Parts:
- C16: value TBD (18p) -> 18p
- C17: value TBD (100n) -> DNP
Changed lines of the file:
@@
 P 12550 4500
 F 0 "C17" H 12642 4546 50  0000 L CNN
-F 1 "TBD (100n)" H 12642 4455 50  0000 L CNN
+F 1 "DNP" H 12642 4455 50  0000 L CNN
 F 2 "Capacitor_SMD:C_0402_1005Metric" H 12550 4500 50  0001 C CNN
 F 3 "~" H 12550 4500 50  0001 C CNN
@@
 P 11500 3950
 F 0 "C16" V 11450 3850 50  0000 C CNN
-F 1 "TBD (18p)" V 11600 3950 50  0000 C CNN
+F 1 "18p" V 11600 3950 50  0000 C CNN
 F 2 "Capacitor_SMD:C_0402_1005Metric" H 11500 3950 50  0001 C CNN
 F 3 "~" H 11500 3950 50  0001 C CNN

Commit message: optimized values
Parts:
- C12, C13, C14, C15: value 1uF -> 1μF 25V
Changed lines of the file:
@@
 AR Path="/5BF2423B" Ref="C15"  Part="1"
 F 0 "C15" H 13865 7996 50  0000 L CNN
-F 1 "1uF" H 13865 7905 50  0000 L CNN
+F 1 "1μF 25V" H 13865 7905 50  0000 L CNN
 F 2 "Capacitor_SMD:C_0402_1005Metric" H 13788 7800 50  0001 C CNN
 F 3 "~" H 13750 7950 50  0001 C CNN
@@
 AR Path="/5BF2BF8E" Ref="C13"  Part="1"
 F 0 "C13" H 13415 7996 50  0000 L CNN
-F 1 "1uF" H 13415 7905 50  0000 L CNN
+F 1 "1μF 25V" H 13415 7905 50  0000 L CNN
 F 2 "Capacitor_SMD:C_0402_1005Metric" H 13338 7800 50  0001 C CNN
 F 3 "~" H 13300 7950 50  0001 C CNN
@@
 AR Path="/5BF7A5D6" Ref="C14"  Part="1"
 F 0 "C14" H 13865 6396 50  0000 L CNN
-F 1 "1uF" H 13865 6305 50  0000 L CNN
+F 1 "1μF 25V" H 13865 6305 50  0000 L CNN
 F 2 "Capacitor_SMD:C_0402_1005Metric" H 13788 6200 50  0001 C CNN
 F 3 "~" H 13750 6350 50  0001 C CNN
@@
 AR Path="/5BF7A6AC" Ref="C12"  Part="1"
 F 0 "C12" H 13365 6696 50  0000 L CNN
-F 1 "1uF" H 13365 6605 50  0000 L CNN
+F 1 "1μF 25V" H 13365 6605 50  0000 L CNN
 F 2 "Capacitor_SMD:C_0402_1005Metric" H 13288 6500 50  0001 C CNN
 F 3 "~" H 13250 6650 50  0001 C CNN

Commit message: added BOM
Other:
- note removed: "Todo:\nDesign auf 4/4 mil\nvias kleiner\nTimer umpfoten"
Changed lines of the file:
@@
 Text GLabel 8050 3300 2    60   Input ~ 0
 PWM
-Text Notes 9450 3600 0    50   ~ 0
-Todo:\nDesign auf 4/4 mil\nvias kleiner\nTimer umpfoten
 $Comp
 L power:+3V3 #PWR0148
