File: KiCAD/C245-Test/C245.sch (KiCad schematic (older format))
At the start: 64 parts, among them J1 USB_C_Receptacle_USB2.0, J2 OLED_64x32, J3 C245, J5 DNP, P1 TC2030-CTX, Q1 SS8050, Q2 DMP3017SFG, SW1 key1, SW2 key2, U1 USBLC6-4SC6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

Commit message: added C245_Test
Parts:
- removed C9: 1μF 25V, otter:C_0603, symbol Device:C
- removed J5: DNP, Resistor_SMD:R_0402_1005Metric, symbol Device:R
- NT1: renamed from NT?; footprint (none) -> NetTie:NetTie-2_SMD_Pad0.5mm
- P1: footprint Tag-Connect:TC2030-NL_SMALL -> otter:TC2030
Connections:
- net at R5.2, U4.44 (BOOT0): now also SW2.2, U4.2 (PC13)
- net at U4.14 (PA4): no longer SW2.2
Other:
- moved on the sheet: SW2
Changed lines of the file:
@@
 $EndDescr
 Wire Wire Line
-	5750 1500 5750 1600
-Wire Wire Line
-	5750 1600 6750 1600
+	5750 1600 6350 1600
 Wire Wire Line
 	7550 4300 7550 4200
@@
 Wire Wire Line
 	8050 3900 8350 3900
-Connection ~ 5750 1600
 Wire Wire Line
 	5750 2000 5750 2100
-Wire Wire Line
-	5750 1100 5750 1200
 Wire Wire Line
 	7250 4300 7250 4400
@@
 F 3 "" H 7250 1000 50  0001 C CNN
 	1    7250 1000
-	1    0    0    -1
-$EndComp
-$Comp
-L power:+3V3 #PWR0102
-U 1 1 5A9AC22A
-P 5750 1100
-F 0 "#PWR0102" H 5750 950 50  0001 C CNN
-F 1 "+3V3" H 5765 1273 50  0000 C CNN
-F 2 "" H 5750 1100 50  0001 C CNN
-F 3 "" H 5750 1100 50  0001 C CNN
-	1    5750 1100
 	1    0    0    -1
 $EndComp
@@
 F 3 "~" H 5650 5150 50  0001 C CNN
 	1    5650 5150
-	1    0    0    -1
-$EndComp
-$Comp
-L Device:C C9
-U 1 1 5A9C1C7E
-P 6150 5150
-F 0 "C9" H 6265 5196 50  0000 L CNN
-F 1 "1μF 25V" H 6265 5105 50  0000 L CNN
-F 2 "otter:C_0603" H 6188 5000 50  0001 C CNN
-F 3 "~" H 6150 5150 50  0001 C CNN
-	1    6150 5150
 	1    0    0    -1
 $EndComp
@@
 F 0 "P1" H 1700 5992 40  0000 C CNN
 F 1 "TC2030-CTX" H 1700 5916 40  0000 C CNN
-F 2 "Tag-Connect:TC2030-NL_SMALL" H 1700 5700 60  0001 C CNN
+F 2 "otter:TC2030" H 1700 5700 60  0001 C CNN
 F 3 "" H 1700 5700 60  0001 C CNN
 	1    1700 5700
@@
 L Switch:SW_Push SW2
 U 1 1 5C1295B7
-P 9500 2500
-F 0 "SW2" V 9454 2648 50  0000 L CNN
-F 1 "key2" V 9545 2648 50  0000 L CNN
-F 2 "Button_Switch_SMD:SW_SPST_EVQP7C" H 9500 2700 50  0001 C CNN
-F 3 "" H 9500 2700 50  0001 C CNN
-	1    9500 2500
+P 5750 1200
+F 0 "SW2" V 5704 1348 50  0000 L CNN
+F 1 "key2" V 5795 1348 50  0000 L CNN
+F 2 "Button_Switch_SMD:SW_SPST_EVQP7C" H 5750 1400 50  0001 C CNN
+F 3 "" H 5750 1400 50  0001 C CNN
+	1    5750 1200
 	0    -1   1    0
 $EndComp
@@
 L power:+3V3 #PWR0142
 U 1 1 5C1295BE
-P 9500 2200
-F 0 "#PWR0142" H 9500 2050 50  0001 C CNN
-F 1 "+3V3" H 9515 2373 50  0000 C CNN
-F 2 "" H 9500 2200 50  0001 C CNN
-F 3 "" H 9500 2200 50  0001 C CNN
-	1    9500 2200
+P 5750 900
+F 0 "#PWR0142" H 5750 750 50  0001 C CNN
+F 1 "+3V3" H 5765 1073 50  0000 C CNN
+F 2 "" H 5750 900 50  0001 C CNN
+F 3 "" H 5750 900 50  0001 C CNN
+	1    5750 900
 	-1   0    0    -1
 $EndComp
 Wire Wire Line
-	9500 2200 9500 2300
+	5750 900  5750 1000
 Wire Wire Line
 	8050 2900 9500 2900
 Wire Wire Line
-	9500 2900 9500 2700
+	5750 1600 5750 1400
 Wire Wire Line
 	10600 3750 10700 3750
@@
 Wire Wire Line
 	9250 7150 9100 7150
-$Comp
-L Device:R J5
-U 1 1 5BE7685C
-P 5750 1350
-F 0 "J5" H 5680 1304 50  0000 R CNN
-F 1 "DNP" H 5680 1395 50  0000 R CNN
-F 2 "Resistor_SMD:R_0402_1005Metric" V 5680 1350 50  0001 C CNN
-F 3 "~" H 5750 1350 50  0001 C CNN
-	1    5750 1350
-	-1   0    0    1
-$EndComp
 $Comp
 L Device:C C6
@@
 $EndComp
 $Comp
-L Device:Net-Tie_2 NT?
+L Device:Net-Tie_2 NT1
 U 1 1 5E6BBB99
 P 15350 4400
-F 0 "NT?" H 15350 4311 50  0000 C CNN
+F 0 "NT1" H 15350 4311 50  0000 C CNN
 F 1 "JUNC_N" H 15350 4220 50  0000 C CNN
-F 2 "" H 15350 4400 50  0001 C CNN
+F 2 "NetTie:NetTie-2_SMD_Pad0.5mm" H 15350 4400 50  0001 C CNN
 F 3 "~" H 15350 4400 50  0001 C CNN
 	1    15350 4400
@@
 AR Path="/588FA3A4/5E6DCFE3" Ref="#PWR?"  Part="1"
 AR Path="/588FD270/5E6DCFE3" Ref="#PWR?"  Part="1"
-AR Path="/5E6DCFE3" Ref="#PWR?"  Part="1"
-F 0 "#PWR?" H 15500 4000 50  0001 C CNN
+AR Path="/5E6DCFE3" Ref="#PWR0149"  Part="1"
+F 0 "#PWR0149" H 15500 4000 50  0001 C CNN
 F 1 "GND" V 15505 4122 50  0000 R CNN
 F 2 "" H 15500 4250 50  0001 C CNN
@@
 Wire Wire Line
 	12550 4400 15250 4400
+Connection ~ 5750 1600
+Wire Wire Line
+	6750 2100 6350 2100
+Wire Wire Line
+	6350 2100 6350 1600
+Connection ~ 6350 1600
+Wire Wire Line
+	6350 1600 6750 1600
 $EndSCHEMATC

Commit message: added C245_Test
Parts:
- added C?: 1μF 25V, otter:C_0603, symbol Device:C
Connections:
- net +3V3: now also C?.1
- net GND: now also C?.2
Other:
- moved on the sheet: C10
Changed lines of the file:
@@
 L Device:C C?
 U 1 1 5BD7CA35
-P 6600 5150
+P 6150 5150
 AR Path="/588FB1D7/5BD7CA35" Ref="C?"  Part="1"
 AR Path="/588FD270/5BD7CA35" Ref="C?"  Part="1"
 AR Path="/5BD7CA35" Ref="C10"  Part="1"
-F 0 "C10" H 6715 5196 50  0000 L CNN
-F 1 "0.1μF" H 6715 5105 50  0000 L CNN
-F 2 "otter:C_0402" H 6638 5000 50  0001 C CNN
-F 3 "~" H 6600 5150 50  0001 C CNN
-	1    6600 5150
+F 0 "C10" H 6265 5196 50  0000 L CNN
+F 1 "0.1μF" H 6265 5105 50  0000 L CNN
+F 2 "otter:C_0402" H 6188 5000 50  0001 C CNN
+F 3 "~" H 6150 5150 50  0001 C CNN
+	1    6150 5150
 	1    0    0    -1
 $EndComp
@@
 Wire Wire Line
 	6350 1600 6750 1600
+$Comp
+L Device:C C?
+U 1 1 5E7E7440
+P 6600 5150
+AR Path="/588FB1D7/5E7E7440" Ref="C?"  Part="1"
+AR Path="/588FD270/5E7E7440" Ref="C?"  Part="1"
+AR Path="/5E7E7440" Ref="C?"  Part="1"
+F 0 "C?" H 6715 5196 50  0000 L CNN
+F 1 "1μF 25V" H 6715 5105 50  0000 L CNN
+F 2 "otter:C_0603" H 6638 5000 50  0001 C CNN
+F 3 "~" H 6600 5150 50  0001 C CNN
+	1    6600 5150
+	1    0    0    -1
+$EndComp
 $EndSCHEMATC

Commit message: added connector pcb, added Gerber
Parts:
- U3: footprint Package_DFN_QFN:QFN-24-1EP_4x4mm_P0.5mm_EP2.7x2.7mm -> otter:QFN-24-1EP_4x4mm_P0.5mm_EP2.7x2.7mm
- gave numbers to parts that had none: 1
Changed lines of the file:
@@
 F 0 "U3" H 4600 7150 50  0000 C CNN
 F 1 "STUSB4500QTR" H 4600 7250 50  0000 C CNN
-F 2 "Package_DFN_QFN:QFN-24-1EP_4x4mm_P0.5mm_EP2.7x2.7mm" H 4300 7900 50  0001 C CNN
+F 2 "otter:QFN-24-1EP_4x4mm_P0.5mm_EP2.7x2.7mm" H 4300 7900 50  0001 C CNN
 F 3 "" H 4300 7900 50  0001 C CNN
 	1    4300 7900
@@
 AR Path="/588FB1D7/5E7E7440" Ref="C?"  Part="1"
 AR Path="/588FD270/5E7E7440" Ref="C?"  Part="1"
-AR Path="/5E7E7440" Ref="C?"  Part="1"
-F 0 "C?" H 6715 5196 50  0000 L CNN
+AR Path="/5E7E7440" Ref="C9"  Part="1"
+F 0 "C9" H 6715 5196 50  0000 L CNN
 F 1 "1μF 25V" H 6715 5105 50  0000 L CNN
 F 2 "otter:C_0603" H 6638 5000 50  0001 C CNN
