File: KiCAD/OtterIron_Devkit/OtterIron_Devkit.sch (KiCad schematic (older format))
At the start: 63 parts, among them J1 USB_C_Receptacle_USB2.0, J2 OLED_64x32, J3 C245, P1 TC2030-CTX, Q1 SS8050, Q2 DMP3017SFG, SW1 key1, SW2 key2, U1 USBLC6-4SC6, U2 AP2204R-3.3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

Commit message: updated files
Parts:
- P1: symbol TS100C-rescue:TC2030-CTX-Tag-Connect-pd-buddy-sink-rescue-usb-c-otter-rescue-usb-c-otter-rescue -> OtterIron_Devkit-rescue:TC2030-CTX-Tag-Connect-pd-buddy-sink-rescue-usb-c-otter-rescue-usb-c-otter-rescue-TS100C-rescue
- Q2: symbol TS100C-rescue:DMP3017SFG-pd-buddy-pd-buddy-sink-rescue-pd-buddy-sink-rescue-usb-c-otter-rescue-usb-c-otter-rescue -> OtterIron_Devkit-rescue:DMP3017SFG-pd-buddy-pd-buddy-sink-rescue-pd-buddy-sink-rescue-usb-c-otter-rescue-usb-c-otter-re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
Changed lines of the file:
@@
 	13600 3050 13600 3150
 $Comp
-L TS100C-rescue:DMP3017SFG-pd-buddy-pd-buddy-sink-rescue-pd-buddy-sink-rescue-usb-c-otter-rescue-usb-c-otter-rescue Q?
+L OtterIron_Devkit-rescue:DMP3017SFG-pd-buddy-pd-buddy-sink-rescue-pd-buddy-sink-rescue-usb-c-otter-rescue-usb-c-otter-rescue-TS100C-rescue Q?
 U 1 1 5BD78C00
 P 14450 3550
@@
 $EndComp
 $Comp
-L TS100C-rescue:TC2030-CTX-Tag-Connect-pd-buddy-sink-rescue-usb-c-otter-rescue-usb-c-otter-rescue P1
+L OtterIron_Devkit-rescue:TC2030-CTX-Tag-Connect-pd-buddy-sink-rescue-usb-c-otter-rescue-usb-c-otter-rescue-TS100C-rescue P1
 U 1 1 5BE3611C
 P 1700 5700
