File: KiCAD/Otter-Iron_Devkit/OtterIron_Devkit.kicad_pcb (KiCad board)
At the start: 2 copper layers, 28 x 30 mm, 64 parts, among them J1 USB_C_Receptacle_USB2.0, J2 OLED_64x32, J3 C245, P1 TC2030-CTX, Q1 SS8050, Q2 DMP3017SFG, SW1 key1, SW2 key2, U1 USBLC6-4SC6, U2 AP2204R-3.3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

Commit message: added v2.0
Parts:
- removed G***: LOGO, otter:OtterIron_Devkit_silk
- added C23: 1000µF, otter:CP_Radial_D10.0mm_P5.00mm_flat, B.Cu at (103.2, 91.5)
- added C24: 1000µF, otter:CP_Radial_D10.0mm_P5.00mm_flat, B.Cu at (93.2, 91.5)
- added L1: 4.7u, otter:Inductor_4040, F.Cu at (91.5, 100.0)
- added Q3: SS8050, Package_TO_SOT_SMD:SOT-23, F.Cu at (92.1, 105.3)
- added Q4: BC807, Package_TO_SOT_SMD:SOT-23, F.Cu at (94.7, 108.0)
- added R25: 2k37, otter:R_0402, F.Cu at (96.5, 110.5)
- R19: footprint otter:R_0402 -> otter:R_0603
- moved R21 17.8 mm to (113.1, 104.8), turned to 90 degrees
- moved R20 16.4 mm to (112.2, 104.8), turned to 270 degrees
- moved R22 15.9 mm to (108.5, 92.0), turned to 180 degrees
- moved U7 15.1 mm to (112.0, 108.7), turned to 0 degrees
- moved R8 14.5 mm to (112.5, 111.0), turned to 180 degrees
- moved C1 11.7 mm to (94.4, 102.3), turned to 270 degrees
- moved C18 11.0 mm to (110.0, 115.9), turned to 180 degrees
- moved R2 9.69 mm to (109.6, 114.5), turned to 270 degrees
- moved C4 8.37 mm to (94.4, 104.8), turned to 90 degrees
- moved R12 7.45 mm to (94.7, 110.2), turned to 0 degrees
- moved U6 6.85 mm to (111.8, 114.2), turned to 180 degrees
- moved U2 6.60 mm to (97.4, 104.0), turned to 0 degrees
- moved Q1 6.41 mm to (98.0, 109.1), turned to 270 degrees
- moved Q2 5.97 mm to (93.0, 95.5)
- moved R9 5.53 mm to (98.4, 106.9), turned to 0 degrees
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Connections:
- J3 pad 5: Net-(D3-Pad1) -> Net-(J3-Pad5)
- R19 pad 1: Net-(Q1-Pad3) -> Net-(Q3-Pad2)
Routing:
- net VBUS: track 50.2 -> 66.8 mm, vias 7 -> 2
- net Net-(D3-Pad1): track 26.4 -> 11.1 mm
- net GND: track 18.2 -> 33.4 mm, vias 56 -> 61
- net Net-(C23-Pad1): track 5.35 -> 19.9 mm
- net Net-(Q3-Pad1): track 0.00 -> 7.49 mm
- net Net-(Q3-Pad2): track 0.00 -> 7.18 mm
- net Net-(Q2-Pad4): track 6.00 -> 12.6 mm
- net PWM: track 15.3 -> 10.5 mm
- net IIN: track 19.3 -> 15.5 mm, vias 2 -> 0
- net +3V3: track 100.1 -> 103.3 mm, vias 6 -> 8
- net UIN: track 13.6 -> 15.3 mm
- net SWDIO: track 14.3 -> 13.1 mm
- net Net-(R21-Pad1): track 1.39 -> 2.51 mm
- net Net-(SW1-Pad2): track 13.2 -> 14.3 mm, vias 0 -> 2
- net TREF: track 2.85 -> 1.84 mm
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- added copper zone on F.Cu, net Net-(J3-Pad5)
Other:
- board text removed: "*mau*"
