File: KiCAD/Otter-Iron_Devkit/OtterIron_Devkit.sch (KiCad schematic (older format))
At the start: 63 parts, among them J1 USB_C_Receptacle_USB2.0, J2 OLED_64x32, J3 C245, P1 TC2030-CTX, Q1 SS8050, Q2 DMP3017SFG, SW1 key1, SW2 key2, U1 USBLC6-4SC6, U2 AP2204R-3.3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

Commit message: added v2.0
Parts:
- added C23, C24: 1000µF, otter:CP_Radial_D10.0mm_P5.00mm_flat, symbol Device:CP_Small
- added L1: 4.7u, otter:Inductor_4040, symbol Device:L
- added Q3: SS8050, Package_TO_SOT_SMD:SOT-23, symbol Transistor_BJT:MMBT3904
- added Q4: BC807, Package_TO_SOT_SMD:SOT-23, symbol Transistor_BJT:BC807
- added R25: 2k37, otter:R_0402, symbol Device:R
- R19: footprint otter:R_0402 -> otter:R_0603
Connections:
- net GND: now also C23.2, C24.2, Q4.3 (C)
- net VBUS: now also Q3.3 (C)
- net at Q2.1 (S), Q2.2 (S), Q2.3 (S)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: now also C23.1, C24.1
- net at D3.1 (K), Q2.5 (D): now also L1.1; no longer J3.5 (Pin_5)
- net at Q1.3 (C), R12.2: now also R25.1; no longer R19.1
- new net: Q3.2 (E), Q4.2 (E), R19.1
- new net: J3.5 (Pin_5), L1.2
- new net: Q3.1 (B), Q4.1 (B), R25.2
Other:
- moved on the sheet: Q1, R12, R19, R9
Changed lines of the file:
@@
 EESchema Schematic File Version 4
+LIBS:OtterIron_Devkit-cache
 EELAYER 30 0
 EELAYER END
@@
 	1    0    0    -1
 $EndComp
-Wire Wire Line
-	13600 4550 13600 4250
-Wire Wire Line
-	13600 3050 13600 3150
 $Comp
 L OtterIron_Devkit-rescue:DMP3017SFG-pd-buddy-pd-buddy-sink-rescue-pd-buddy-sink-rescue-usb-c-otter-rescue-usb-c-otter-rescue-TS100C-rescue Q?
@@
 L power:VBUS #PWR?
 U 1 1 5BD78C13
-P 13600 3050
+P 12950 3100
 AR Path="/588FA3A4/5BD78C13" Ref="#PWR?"  Part="1"
 AR Path="/588FD270/5BD78C13" Ref="#PWR?"  Part="1"
 AR Path="/5BD78C13" Ref="#PWR0112"  Part="1"
-F 0 "#PWR0112" H 13600 2900 50  0001 C CNN
-F 1 "VBUS" H 13615 3223 50  0000 C CNN
-F 2 "" H 13600 3050 50  0001 C CNN
-F 3 "" H 13600 3050 50  0001 C CNN
-	1    13600 3050
+F 0 "#PWR0112" H 12950 2950 50  0001 C CNN
+F 1 "VBUS" H 12965 3273 50  0000 C CNN
+F 2 "" H 12950 3100 50  0001 C CNN
+F 3 "" H 12950 3100 50  0001 C CNN
+	1    12950 3100
 	1    0    0    -1
 $EndComp
@@
 L power:GND #PWR?
 U 1 1 5BD78C25
-P 13600 4550
+P 12950 3900
 AR Path="/588FA3A4/5BD78C25" Ref="#PWR?"  Part="1"
 AR Path="/588FD270/5BD78C25" Ref="#PWR?"  Part="1"
 AR Path="/5BD78C25" Ref="#PWR0114"  Part="1"
-F 0 "#PWR0114" H 13600 4300 50  0001 C CNN
-F 1 "GND" H 13605 4377 50  0000 C CNN
-F 2 "" H 13600 4550 50  0001 C CNN
-F 3 "" H 13600 4550 50  0001 C CNN
-	1    13600 4550
+F 0 "#PWR0114" H 12950 3650 50  0001 C CNN
+F 1 "GND" H 12955 3727 50  0000 C CNN
+F 2 "" H 12950 3900 50  0001 C CNN
+F 3 "" H 12950 3900 50  0001 C CNN
+	1    12950 3900
 	1    0    0    -1
 $EndComp
@@
 L Device:R R?
 U 1 1 5BD78C38
-P 13600 3300
+P 12950 3250
 AR Path="/588FA3A4/5BD78C38" Ref="R?"  Part="1"
 AR Path="/588FD270/5BD78C38" Ref="R?"  Part="1"
 AR Path="/5BD78C38" Ref="R12"  Part="1"
-F 0 "R12" H 13670 3346 50  0000 L CNN
-F 1 "2k37" H 13670 3255 50  0000 L CNN
-F 2 "otter:R_0402" V 13530 3300 50  0001 C CNN
-F 3 "~" H 13600 3300 50  0001 C CNN
-	1    13600 3300
+F 0 "R12" H 13020 3296 50  0000 L CNN
+F 1 "2k37" H 13020 3205 50  0000 L CNN
+F 2 "otter:R_0402" V 12880 3250 50  0001 C CNN
+F 3 "~" H 12950 3250 50  0001 C CNN
+	1    12950 3250
 	1    0    0    -1
 $EndComp
@@
 L Device:R R?
 U 1 1 5BD78C3F
-P 13150 4050
+P 12500 3700
 AR Path="/588FA3A4/5BD78C3F" Ref="R?"  Part="1"
 AR Path="/588FD270/5BD78C3F" Ref="R?"  Part="1"
 AR Path="/5BD78C3F" Ref="R9"  Part="1"
-F 0 "R9" V 12943 4050 50  0000 C CNN
-F 1 "2k37" V 13034 4050 50  0000 C CNN
-F 2 "otter:R_0402" V 13080 4050 50  0001 C CNN
-F 3 "~" H 13150 4050 50  0001 C CNN
-	1    13150 4050
+F 0 "R9" V 12293 3700 50  0000 C CNN
+F 1 "2k37" V 12384 3700 50  0000 C CNN
+F 2 "otter:R_0402" V 12430 3700 50  0001 C CNN
+F 3 "~" H 12500 3700 50  0001 C CNN
+	1    12500 3700
 	0    -1   1    0
 $EndComp
@@
 L Transistor_BJT:MMBT3904 Q?
 U 1 1 5BD78C4D
-P 13500 4050
+P 12850 3700
 AR Path="/588FA3A4/5BD78C4D" Ref="Q?"  Part="1"
 AR Path="/588FD270/5BD78C4D" Ref="Q?"  Part="1"
 AR Path="/5BD78C4D" Ref="Q1"  Part="1"
-F 0 "Q1" H 13691 4096 50  0000 L CNN
-F 1 "SS8050" H 13691 4005 50  0000 L CNN
-F 2 "Package_TO_SOT_SMD:SOT-23" H 13700 3975 50  0001 L CIN
-F 3 "https://www.fairchildsemi.com/datasheets/2N/2N3904.pdf" H 13500 4050 50  0001 L CNN
-	1    13500 4050
+F 0 "Q1" H 13040 3746 50  0000 L CNN
+F 1 "SS8050" H 13040 3655 50  0000 L CNN
+F 2 "Package_TO_SOT_SMD:SOT-23" H 13050 3625 50  0001 L CIN
+F 3 "https://www.fairchildsemi.com/datasheets/2N/2N3904.pdf" H 12850 3700 50  0001 L CNN
+	1    12850 3700
 	1    0    0    -1
 $EndComp
@@
 	1    0    0    -1
 $EndComp
-Text GLabel 13000 4050 0    60   Input ~ 0
+Text GLabel 12350 3700 0    60   Input ~ 0
 PWM
 Text GLabel 5100 3500 0    60   Input ~ 0
@@
 Text GLabel 11400 7450 2    60   Input ~ 0
 TREF
-Wire Wire Line
-	13600 3450 13600 3550
 $Comp
 L Device:R R?
 U 1 1 5C10E2D1
-P 13950 3550
+P 14100 3550
 AR Path="/588FA3A4/5C10E2D1" Ref="R?"  Part="1"
 AR Path="/588FD270/5C10E2D1" Ref="R?"  Part="1"
 AR Path="/5C10E2D1" Ref="R19"  Part="1"
-F 0 "R19" V 13743 3550 50  0000 C CNN
-F 1 "20" V 13834 3550 50  0000 C CNN
-F 2 "otter:R_0402" V 13880 3550 50  0001 C CNN
-F 3 "~" H 13950 3550 50  0001 C CNN
-	1    13950 3550
+F 0 "R19" V 13893 3550 50  0000 C CNN
+F 1 "20" V 13984 3550 50  0000 C CNN
+F 2 "otter:R_0603" V 14030 3550 50  0001 C CNN
+F 3 "~" H 14100 3550 50  0001 C CNN
+	1    14100 3550
 	0    -1   1    0
 $EndComp
 Wire Wire Line
-	14100 3550 14250 3550
-Wire Wire Line
-	13600 3550 13800 3550
-Connection ~ 13600 3550
-Wire Wire Line
-	13600 3550 13600 3850
+	12950 3450 13150 3450
 $Comp
 L Switch:SW_Push SW2
@@
 	14250 2300 14200 2300
 Wire Wire Line
-	14550 2300 14550 3350
+	14550 2300 14550 2650
 Connection ~ 14550 2300
 Wire Wire Line
@@
 	12850 4600 12550 4600
 Connection ~ 12550 4600
-Wire Wire Line
-	14550 3750 14550 3850
-Connection ~ 14550 3850
-Wire Wire Line
-	14550 3850 14550 3950
-Wire Wire Line
-	14550 3850 15650 3850
 $Comp
 L MCU_ST_STM32F0:STM32F072C8Tx U4
@@
 	1    0    0    -1
 $EndComp
+$Comp
+L Device:CP_Small C23
+U 1 1 5E94E082
+P 14850 2900
+F 0 "C23" H 14938 2946 50  0000 L CNN
+F 1 "1000µF" H 14938 2855 50  0000 L CNN
+F 2 "otter:CP_Radial_D10.0mm_P5.00mm_flat" H 14850 2900 50  0001 C CNN
+F 3 "~" H 14850 2900 50  0001 C CNN
+	1    14850 2900
+	1    0    0    -1
+$EndComp
+$Comp
+L Device:CP_Small C24
+U 1 1 5E963268
+P 15400 2900
+F 0 "C24" H 15488 2946 50  0000 L CNN
+F 1 "1000µF" H 15488 2855 50  0000 L CNN
+F 2 "otter:CP_Radial_D10.0mm_P5.00mm_flat" H 15400 2900 50  0001 C CNN
+F 3 "~" H 15400 2900 50  0001 C CNN
+	1    15400 2900
+	1    0    0    -1
+$EndComp
+$Comp
+L power:GND #PWR0102
+U 1 1 5E96DE3A
+P 15400 3000
+F 0 "#PWR0102" H 15400 2750 50  0001 C CNN
+F 1 "GND" H 15405 2827 50  0000 C CNN
+F 2 "" H 15400 3000 50  0001 C CNN
+F 3 "" H 15400 3000 50  0001 C CNN
+	1    15400 3000
+	1    0    0    -1
+$EndComp
+$Comp
+L power:GND #PWR0150
+U 1 1 5E9703E7
+P 14850 3000
+F 0 "#PWR0150" H 14850 2750 50  0001 C CNN
+F 1 "GND" H 14855 2827 50  0000 C CNN
+F 2 "" H 14850 3000 50  0001 C CNN
+F 3 "" H 14850 3000 50  0001 C CNN
+	1    14850 3000
+	1    0    0    -1
+$EndComp
+Wire Wire Line
+	15400 2800 15400 2650
+Wire Wire Line
+	15400 2650 14850 2650
+Wire Wire Line
+	14850 2800 14850 2650
+Connection ~ 14850 2650
+Wire Wire Line
+	14850 2650 14550 2650
+Connection ~ 14550 2650
+Wire Wire Line
+	14550 2650 14550 3350
+Wire Wire Line
+	12950 3500 12950 3450
+Wire Wire Line
+	12950 3400 12950 3450
+Connection ~ 12950 3450
+$Comp
+L Transistor_BJT:MMBT3904 Q?
+U 1 1 5E9C7C2F
+P 13750 3200
+AR Path="/588FA3A4/5E9C7C2F" Ref="Q?"  Part="1"
+AR Path="/588FD270/5E9C7C2F" Ref="Q?"  Part="1"
+AR Path="/5E9C7C2F" Ref="Q3"  Part="1"
+F 0 "Q3" H 13941 3246 50  0000 L CNN
+F 1 "SS8050" H 13941 3155 50  0000 L CNN
+F 2 "Package_TO_SOT_SMD:SOT-23" H 13950 3125 50  0001 L CIN
+F 3 "https://www.fairchildsemi.com/datasheets/2N/2N3904.pdf" H 13750 3200 50  0001 L CNN
+	1    13750 3200
+	1    0    0    -1
+$EndComp
+$Comp
+L Device:R R?
+U 1 1 5E9D3B53
+P 13300 3450
+AR Path="/588FA3A4/5E9D3B53" Ref="R?"  Part="1"
+AR Path="/588FD270/5E9D3B53" Ref="R?"  Part="1"
+AR Path="/5E9D3B53" Ref="R25"  Part="1"
+F 0 "R25" V 13185 3450 50  0000 C CNN
+F 1 "2k37" V 13094 3450 50  0000 C CNN
+F 2 "otter:R_0402" V 13230 3450 50  0001 C CNN
+F 3 "~" H 13300 3450 50  0001 C CNN
+	1    13300 3450
+	0    -1   -1   0
+$EndComp
+$Comp
+L Transistor_BJT:BC807 Q4
+U 1 1 5E9F3988
+P 13750 3900
+F 0 "Q4" H 13941 3854 50  0000 L CNN
+F 1 "BC807" H 13941 3945 50  0000 L CNN
+F 2 "Package_TO_SOT_SMD:SOT-23" H 13950 3825 50  0001 L CIN
+F 3 "http://www.fairchildsemi.com/ds/BC/BC807.pdf" H 13750 3900 50  0001 L CNN
+	1    13750 3900
+	1    0    0    1
+$EndComp
+Wire Wire Line
+	13950 3550 13850 3550
+Wire Wire Line
+	13850 3550 13850 3400
+Wire Wire Line
+	13850 3700 13850 3550
+Connection ~ 13850 3550
+Wire Wire Line
+	13550 3200 13550 3450
+Wire Wire Line
+	13450 3450 13550 3450
+Connection ~ 13550 3450
+Wire Wire Line
+	13550 3450 13550 3900
+$Comp
+L power:VBUS #PWR?
+U 1 1 5EA54D82
+P 13850 3000
+AR Path="/588FA3A4/5EA54D82" Ref="#PWR?"  Part="1"
+AR Path="/588FD270/5EA54D82" Ref="#PWR?"  Part="1"
+AR Path="/5EA54D82" Ref="#PWR0151"  Part="1"
+F 0 "#PWR0151" H 13850 2850 50  0001 C CNN
+F 1 "VBUS" H 13865 3173 50  0000 C CNN
+F 2 "" H 13850 3000 50  0001 C CNN
+F 3 "" H 13850 3000 50  0001 C CNN
+	1    13850 3000
+	1    0    0    -1
+$EndComp
+$Comp
+L power:GND #PWR0152
+U 1 1 5EA61605
+P 13850 4100
+F 0 "#PWR0152" H 13850 3850 50  0001 C CNN
+F 1 "GND" H 13855 3927 50  0000 C CNN
+F 2 "" H 13850 4100 50  0001 C CNN
+F 3 "" H 13850 4100 50  0001 C CNN
+	1    13850 4100
+	1    0    0    -1
+$EndComp
+Wire Wire Line
+	14550 3750 14550 3850
+$Comp
+L Device:L L1
+U 1 1 5E95244D
+P 15150 3850
+F 0 "L1" V 15340 3850 50  0000 C CNN
+F 1 "4.7u" V 15249 3850 50  0000 C CNN
+F 2 "otter:Inductor_4040" H 15150 3850 50  0001 C CNN
+F 3 "~" H 15150 3850 50  0001 C CNN
+	1    15150 3850
+	0    -1   -1   0
+$EndComp
+Wire Wire Line
+	15300 3850 15650 3850
+Wire Wire Line
+	15000 3850 14550 3850
+Connection ~ 14550 3850
+Wire Wire Line
+	14550 3850 14550 3950
 $EndSCHEMATC
