File: KiCAD/Otter-Iron_Devkit/C245_conn/C245_conn.sch (KiCad schematic (older format))
At the start: 2 parts, among them J1 Otter-Iron, J2 C245

Commit message: added v2.0
Parts:
- added C1: 10u, Capacitor_SMD:C_1206_3216Metric, symbol Device:C
- J1: footprint Connector_PinHeader_2.54mm:PinHeader_1x06_P2.54mm_Horizontal -> Connector_PinHeader_2.54mm:PinHeader_1x06_P2.54mm_Vertical
Connections:
- net GND: now also C1.2
- net HEAT: now also C1.1
Changed lines of the file:
@@
 EESchema Schematic File Version 4
+LIBS:C245_conn-cache
 EELAYER 30 0
 EELAYER END
@@
 F 0 "J1" H 6922 3082 50  0000 R CNN
 F 1 "Otter-Iron" H 6922 3173 50  0000 R CNN
-F 2 "Connector_PinHeader_2.54mm:PinHeader_1x06_P2.54mm_Horizontal" H 6950 3200 50  0001 C CNN
+F 2 "Connector_PinHeader_2.54mm:PinHeader_1x06_P2.54mm_Vertical" H 6950 3200 50  0001 C CNN
 F 3 "~" H 6950 3200 50  0001 C CNN
 	1    6950 3200
@@
 Text GLabel 8000 3100 0    50   Input ~ 0
 HEAT
+Text GLabel 7650 2750 2    50   Input ~ 0
+HEAT
+$Comp
+L power:GND #PWR0103
+U 1 1 5E939CFD
+P 7350 2750
+F 0 "#PWR0103" H 7350 2500 50  0001 C CNN
+F 1 "GND" V 7355 2622 50  0000 R CNN
+F 2 "" H 7350 2750 50  0001 C CNN
+F 3 "" H 7350 2750 50  0001 C CNN
+	1    7350 2750
+	0    1    1    0
+$EndComp
+$Comp
+L Device:C C1
+U 1 1 5E939EB4
+P 7500 2750
+F 0 "C1" V 7248 2750 50  0000 C CNN
+F 1 "10u" V 7339 2750 50  0000 C CNN
+F 2 "Capacitor_SMD:C_1206_3216Metric" H 7538 2600 50  0001 C CNN
+F 3 "~" H 7500 2750 50  0001 C CNN
+	1    7500 2750
+	0    1    1    0
+$EndComp
 $EndSCHEMATC
