File: KiCAD/Otter-Iron/TS100C.kicad_pcb (KiCad board)
At the start: 4 copper layers, 84 x 10 mm, 64 parts, among them J1 USB_C_Receptacle_USB2.0, J2 OLED_64x32, J3 A, J4 B, J5 DNP, P1 TC2030-CTX, Q1 SS8050, Q2 DMP3017SFG, SW1 key1, SW2 key2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

Commit message: hw v2.4 released
Other:
- net class Default removed
- board text added: "Design by: @_Jana_Marie"
- board text removed: "Design by: JanHenrik"
